Commit message: add gnss

File: urdf/vitulus4WD_description.urdf.xacro (robot description, xacro)
@@ -161,5 +161,6 @@
             add_plug="$(arg add_plug)"
             use_mesh="$(arg use_mesh)">
-        <origin xyz="0.222 0 0.280" rpy="0 0 ${deg_to_rad*0}"/>
+<!--        <origin xyz="0.222 0 0.280" rpy="0 0 ${deg_to_rad*0}"/>-->
+        <origin xyz="0.202 0.024 0.280" rpy="0 0 ${deg_to_rad*0}"/>
     </xacro:sensor_d435>
   <link name="t265_link">
@@ -171,3 +172,31 @@
       <origin xyz="0.232 0 0.322" rpy="${deg_to_rad*90} 0 ${deg_to_rad*270}"/>
     </joint>
+    <!-- GNSS UBLOX -->
+   <link name="gnss_heading">
+    <visual>
+        <geometry>
+            <box size="0.01 0.01 0.01" />
+          </geometry>
+        <origin rpy="0 0 0" xyz="0 0 0"/>
+    </visual>
+  </link>
+  <joint name="gnss_heading_joint" type="fixed">
+    <parent link="base_link"/>
+    <child link="gnss"/>
+    <origin xyz="-0.16 -0.21 0.3" rpy="0 0 -1.5707963"/>
+  </joint>
+  <link name="gnss">
+    <visual>
+        <geometry>
+            <box size="0.01 0.01 0.01" />
+          </geometry>
+        <origin rpy="0 0 0" xyz="0 0 0"/>
+    </visual>
+  </link>
+  <joint name="gnss_joint" type="fixed">
+    <parent link="base_link"/>
+    <child link="gnsslite"/>
+    <!-- origin xyz="-0.16 0.21 0.3" rpy="0 0 -1.5707963"/ -->
+    <origin xyz="-0.16 0.21 0.3" rpy="0 0 -1.5707963"/>
+  </joint>
 </robot>

Commit message: add gnss

File: urdf/vitulus4WD_description.urdf.xacro (robot description, xacro)
@@ -183,5 +183,5 @@
   <joint name="gnss_heading_joint" type="fixed">
     <parent link="base_link"/>
-    <child link="gnss"/>
+    <child link="gnss_heading"/>
     <origin xyz="-0.16 -0.21 0.3" rpy="0 0 -1.5707963"/>
   </joint>
@@ -196,5 +196,5 @@
   <joint name="gnss_joint" type="fixed">
     <parent link="base_link"/>
-    <child link="gnsslite"/>
+    <child link="gnss"/>
     <!-- origin xyz="-0.16 0.21 0.3" rpy="0 0 -1.5707963"/ -->
     <origin xyz="-0.16 0.21 0.3" rpy="0 0 -1.5707963"/>

Commit message: imu rear

File: urdf/vitulus4WD_description.urdf.xacro (robot description, xacro)
@@ -101,5 +101,18 @@
 <!--    <origin xyz="0.164 0.0025 0.297" rpy="0 0 0"/>-->
   </joint>
-    <link name="bno_imu_link">
+<link name="bno_imu_link">
+    <visual>
+        <geometry>
+            <box size="0.01 0.01 0.01" />
+          </geometry>
+        <origin rpy="0 0 0" xyz="0 0 0"/>
+    </visual>
+  </link>
+  <joint name="bno_imu_joint" type="fixed">
+    <parent link="chassis"/>
+    <child link="bno_imu_link"/>
+    <origin xyz="-0.20 -0.02 0.3" rpy="0 0 0"/>
+  </joint>
+<!--    <link name="bno_imu_link">
     <visual>
         <geometry>
@@ -113,6 +126,5 @@
     <child link="bno_imu_link"/>
     <origin xyz="-0.03 0.00 0.3" rpy="0 0 0"/>
-<!--    <origin xyz="0.164 0.0025 0.297" rpy="0 0 0"/>-->
-  </joint>
+  </joint>-->
      <link name="mag_link">
     <visual>

Commit message: RplidarC1

File: urdf/vitulus4WD_description.urdf.xacro (robot description, xacro)
@@ -4,5 +4,5 @@
     <xacro:arg name="add_plug" default="false" />
     <xacro:arg name="use_mesh" default="true" />
-    <xacro:include filename="$(find realsense2_description)/urdf/_d435.urdf.xacro" />
+    <xacro:include filename="$(find vitulus_description)/urdf/_d435.urdf.xacro" />
     <xacro:include filename="$(find vitulus_description)/urdf/macros.xacro" />
     <xacro:arg name="laser_visual" default="false"/>
@@ -165,5 +165,5 @@
       <parent link="chassis"/>
       <child link="base_scan"/>
-      <origin xyz="0.079 0 0.348" rpy="0 0 ${deg_to_rad*270}"/>
+      <origin xyz="0.062 0 0.348" rpy="0 0 ${deg_to_rad*270}"/>
     </joint>
     <xacro:sensor_d435
