Commit message: d435 mount: measured pitch trim -1.4 deg
Ground-plane fit on flat concrete showed the depth-reconstructed ground
tilting -1.9 deg with distance (dz/dx -0.033 m/m, 2 mm residual). Two
measurement iterations: -1.8 -> +0.34 deg overcorrection, -1.4 -> -0.13
deg pitch / -0.02 deg roll, plane residual 0.017 m over 651k pts.

File: urdf/vitulus4WD_description.urdf.xacro (robot description, xacro)
@@ -174,5 +174,5 @@
             use_mesh="$(arg use_mesh)">
 <!--        <origin xyz="0.222 0 0.280" rpy="0 0 ${deg_to_rad*0}"/>-->
-        <origin xyz="0.202 0.024 0.280" rpy="0 0 ${deg_to_rad*0}"/>
+        <origin xyz="0.202 0.024 0.280" rpy="0 ${deg_to_rad*-1.4} 0"/>
     </xacro:sensor_d435>
   <link name="t265_link">
